File: kicad/mainboard/mainboard.kicad_sch (KiCad schematic)
At the start: 3 parts

Commit message: Tiny fixups on mainboard: mounting holes and one audio jack
Parts:
- H1, H2, H3: footprint MountingHole:MountingHole_2.7mm_M2.5 -> MountingHole:MountingHole_2.5mm
Changed lines of the file:
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@@
       (effects (font (size 1.27 1.27)) (justify left))
     )
-    (property "Footprint" "MountingHole:MountingHole_2.7mm_M2.5" (id 2) (at 41.91 153.67 0)
+    (property "Footprint" "MountingHole:MountingHole_2.5mm" (id 2) (at 41.91 153.67 0)
       (effects (font (size 1.27 1.27)) hide)
     )
@@
       (effects (font (size 1.27 1.27)) (justify left))
     )
-    (property "Footprint" "MountingHole:MountingHole_2.7mm_M2.5" (id 2) (at 41.91 158.75 0)
+    (property "Footprint" "MountingHole:MountingHole_2.5mm" (id 2) (at 41.91 158.75 0)
       (effects (font (size 1.27 1.27)) hide)
     )
@@
       (effects (font (size 1.27 1.27)) (justify left))
     )
-    (property "Footprint" "MountingHole:MountingHole_2.7mm_M2.5" (id 2) (at 41.91 148.59 0)
+    (property "Footprint" "MountingHole:MountingHole_2.5mm" (id 2) (at 41.91 148.59 0)
       (effects (font (size 1.27 1.27)) hide)
     )
@@
     )
     (path "/cd39498c-2e8a-48dc-a12c-d027bca333f6"
-      (reference "H1") (unit 1) (value "MountingHole") (footprint "MountingHole:MountingHole_2.7mm_M2.5")
+      (reference "H1") (unit 1) (value "MountingHole") (footprint "MountingHole:MountingHole_2.5mm")
     )
     (path "/52826be8-8e78-4f3e-ae6f-41daa025d4c3"
-      (reference "H2") (unit 1) (value "MountingHole") (footprint "MountingHole:MountingHole_2.7mm_M2.5")
+      (reference "H2") (unit 1) (value "MountingHole") (footprint "MountingHole:MountingHole_2.5mm")
     )
     (path "/95be1109-74d2-4230-ac0d-36359fb1c897"
-      (reference "H3") (unit 1) (value "MountingHole") (footprint "MountingHole:MountingHole_2.7mm_M2.5")
+      (reference "H3") (unit 1) (value "MountingHole") (footprint "MountingHole:MountingHole_2.5mm")
     )
     (path "/7dcd6303-5acd-4a81-8a26-a2e196b6bba9/1a96594a-9dc8-4b3b-8e26-65367a600fdd"
